File: hardware/rgb-button-bricklet.kicad_pcb (KiCad board)
At the start: 2 copper layers, 25 x 25 mm, 25 parts, among them P1 CON-SENSOR, P2 Boot, SW1 RGB_SWITCH_AD, U1 XMC1XXX24, U2 DRILL, U3 DRILL, U4 DRILL, U5 DRILL

Commit message: add status led description text
Other:
- board text added: "status"
Changed lines of the file:
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@@
-(kicad_pcb (version 4) (host pcbnew 4.0.7-e1-6374~58~ubuntu17.04.1)
+(kicad_pcb (version 4) (host pcbnew 4.0.7-e2-6376~58~ubuntu17.04.1)
   (general
     (links 41)
@@
     (area 138.344999 89.044999 278.84286 159.815)
     (thickness 1.6)
-    (drawings 12)
+    (drawings 13)
     (tracks 141)
     (zones 0)
@@
     (35 F.Paste user)
     (36 B.SilkS user)
-    (37 F.SilkS user hide)
+    (37 F.SilkS user)
     (38 B.Mask user)
     (39 F.Mask user)
@@
       (net 11 "Net-(R2-Pad2)"))
   )
+  (gr_text status (at 160.45 97.55 90) (layer F.SilkS)
+    (effects (font (size 0.8 0.8) (thickness 0.15)))
+  )
   (gr_text "RGB LED Button\n1.0" (at 141.85 102.4 90) (layer B.SilkS)

Commit message: specify processor
Parts:
- U1: value XMC1XXX24 -> XMC1100-16
Changed lines of the file:
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@@
     (company "Tinkerforge GmbH")
     (comment 1 "Licensed under CERN OHL v.1.1")
-    (comment 2 "Copyright (©) 2017, L.Lauer <lukas@tinkerforge.com>")
+    (comment 2 "Copyright (©) 2017, B.Nordmeyer <bastian@tinkerforge.com>")
   )
   (layers
@@
       (effects (font (size 0.3 0.3) (thickness 0.075)))
     )
-    (fp_text value XMC1XXX24 (at 0 0.8 180) (layer F.Fab)
+    (fp_text value XMC1100-16 (at 0 0.8 180) (layer F.Fab)
       (effects (font (size 0.3 0.3) (thickness 0.075)))
     )
